File: v2.0 Main.brd (EAGLE design)
At the start: 100 x 69.3 mm, 39 parts, among them IC2 PCF8574D, K1 G5LE, Q1 XTAL 16MHz, Q3 Mosfet-N, U1 ARDUINOSPI-REFRENCE, U2 POWER-POD 5V0, U3 ATMEGA328P-MU, U4 POWER-POD 3V3, U7 POWER-POD 5V0

Commit message: Tweaks and berbers
Parts:
- added JP4, JP7, JP9: FIDUCIAL1X2.5-STOP, CISECO eaglecad designs:FIDUCIAL-1X2.5-STOP
