File: v2.0 Main.sch (EAGLE design)
At the start: 39 parts, among them IC2 PCF8574D, K1 G5LE, Q1 XTAL 16MHz, Q3 Mosfet-N, U1 ARDUINOSPI-REFRENCE, U2 POWER-POD 5V0, U3 ATMEGA328P-MU, U4 POWER-POD 3V3, U7 POWER-POD 5V0

Commit message: Tweaks and berbers
Parts:
- added JP4, JP7, JP9: FIDUCIAL1X2.5-STOP, CISECO eaglecad designs:FIDUCIAL1X2.5-STOP
Changed lines of the file:
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@@
 <part name="JP10" library="CISECO eaglecad designs" deviceset="M10" device="LOCK"/>
 <part name="C11" library="rcl" deviceset="CPOL-EU" device="C" value="C 100uF 6.3V"/>
+<part name="JP4" library="CISECO eaglecad designs" deviceset="FIDUCIAL" device="1X2.5-STOP"/>
+<part name="JP7" library="CISECO eaglecad designs" deviceset="FIDUCIAL" device="1X2.5-STOP"/>
+<part name="JP9" library="CISECO eaglecad designs" deviceset="FIDUCIAL" device="1X2.5-STOP"/>
 </parts>
 <sheets>
@@
 <attribute name="VALUE" x="163.703" y="152.8826" size="1.778" layer="96" rot="R270"/>
 </instance>
+<instance part="JP4" gate="G$1" x="220.98" y="22.86"/>
+<instance part="JP7" gate="G$1" x="223.52" y="22.86"/>
+<instance part="JP9" gate="G$1" x="226.06" y="22.86"/>
 </instances>
 <busses>
