File: v2.0 Door.brd (EAGLE design)
At the start: 116 x 48 mm, 18 parts, among them IC1 PCF8574D, Q2 Mosfet-N, U5 ERM2002-1

Commit message: Tweaks and berbers
Parts:
- added JP1, JP2, JP3: FIDUCIAL1X2.5-STOP, CISECO eaglecad designs:FIDUCIAL-1X2.5-STOP
Changed lines of the file:
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@@
 <setting verticaltext="up"/>
 </settings>
-<grid distance="1" unitdist="mm" unit="mm" style="lines" multiple="1" display="yes" altdistance="0.5" altunitdist="mm" altunit="mm"/>
+<grid distance="5" unitdist="mm" unit="mm" style="lines" multiple="1" display="yes" altdistance="2.5" altunitdist="mm" altunit="mm"/>
 <layers>
 <layer number="1" name="Top" color="4" fill="1" visible="yes" active="yes"/>
@@
 <plain>
 <rectangle x1="27" y1="7" x2="87" y2="47" layer="202"/>
-<text x="1.9" y="44.7" size="1.778" layer="21" font="vector" ratio="15">HSNOTTS Gatekeeper</text>
+<text x="7.9" y="45.7" size="1.778" layer="21" font="vector" ratio="15">HSNOTTS Gatekeeper</text>
 <wire x1="114" y1="0" x2="2" y2="0" width="0.15" layer="20"/>
 <wire x1="2" y1="0" x2="0" y2="2" width="0.15" layer="20" curve="-90"/>
@@
 <wire x1="116" y1="46" x2="116" y2="2" width="0.15" layer="20"/>
 <wire x1="116" y1="2" x2="114" y2="0" width="0.15" layer="20" curve="-90"/>
-<text x="31.9" y="44.7" size="1.778" layer="21" font="vector" ratio="15">v2.0</text>
+<text x="7.9" y="42.7" size="1.778" layer="21" font="vector" ratio="15">v2.0</text>
 <text x="81.25" y="8.5" size="1.016" layer="21" ratio="15" rot="R90" align="center-left">Bell</text>
 <text x="86.75" y="8.5" size="1.016" layer="21" ratio="15" rot="R90" align="center-left">Buzzer</text>
@@
 <element name="R10" library="CISECO eaglecad designs" package="R0402-SMALLER" value="0402 10K" x="15.25" y="4" rot="R90"/>
 <element name="L2" library="CISECO eaglecad designs" package="LED5MM" value="LED-BI-COLOUR-5MM" x="19.25" y="5" rot="MR270"/>
+<element name="JP1" library="CISECO eaglecad designs" package="FIDUCIAL-1X2.5-STOP" value="FIDUCIAL1X2.5-STOP" x="3" y="3"/>
+<element name="JP2" library="CISECO eaglecad designs" package="FIDUCIAL-1X2.5-STOP" value="FIDUCIAL1X2.5-STOP" x="97.5" y="15"/>
+<element name="JP3" library="CISECO eaglecad designs" package="FIDUCIAL-1X2.5-STOP" value="FIDUCIAL1X2.5-STOP" x="100" y="40"/>
 </elements>
 <signals>
@@
 <via x="5" y="5" extent="1-16" drill="0.5"/>
 <via x="5" y="10" extent="1-16" drill="0.5"/>
-<via x="5" y="15" extent="1-16" drill="0.5"/>
 <via x="5" y="20" extent="1-16" drill="0.5"/>
 <via x="5" y="25" extent="1-16" drill="0.5"/>
@@
 <via x="5" y="35" extent="1-16" drill="0.5"/>
 <via x="5" y="40" extent="1-16" drill="0.5"/>
-<via x="5" y="45" extent="1-16" drill="0.5"/>
 <via x="10" y="45" extent="1-16" drill="0.5"/>
 <via x="30" y="45" extent="1-16" drill="0.5"/>

Commit message: Update connectors
Parts:
- JP7, JP9: device CISECO eaglecad designs:1X02_LOCK -> CISECO eaglecad designs:MOLEX-1X2_LOCK
- moved JP9 0.50 mm to (80.8, 4.23)
Changed lines of the file:
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@@
 <setting verticaltext="up"/>
 </settings>
-<grid distance="5" unitdist="mm" unit="mm" style="lines" multiple="1" display="yes" altdistance="2.5" altunitdist="mm" altunit="mm"/>
+<grid distance="0.5" unitdist="mm" unit="mm" style="lines" multiple="1" display="yes" altdistance="0.25" altunitdist="mm" altunit="mm"/>
 <layers>
 <layer number="1" name="Top" color="4" fill="1" visible="yes" active="yes"/>
@@
 <element name="R8" library="CISECO eaglecad designs" package="R0402-SMALLER" value="0402 10K" x="107.524" y="39.844"/>
 <element name="Q2" library="TiLDA Mk2 Parts" package="SOT23-3" value="Mosfet-N" x="107.524" y="41.844"/>
-<element name="JP7" library="CISECO eaglecad designs" package="1X02_LOCK" value="" x="86.81" y="4.23" rot="R90"/>
-<element name="JP9" library="CISECO eaglecad designs" package="1X02_LOCK" value="" x="81.27" y="4.23" rot="R90"/>
+<element name="JP7" library="CISECO eaglecad designs" package="MOLEX-1X2_LOCK" value="" x="86.81" y="4.23" rot="R90"/>
+<element name="JP9" library="CISECO eaglecad designs" package="MOLEX-1X2_LOCK" value="" x="80.77" y="4.23" rot="R90"/>
 <element name="R9" library="CISECO eaglecad designs" package="R0402-SMALLER" value="0402 10K" x="15.25" y="6" rot="R90"/>
 <element name="R10" library="CISECO eaglecad designs" package="R0402-SMALLER" value="0402 10K" x="15.25" y="4" rot="R90"/>
@@
 <wire x1="84.5" y1="2" x2="83.5" y2="3" width="0.254" layer="16"/>
 <wire x1="83.5" y1="3" x2="83.5" y2="5.5" width="0.254" layer="16"/>
-<wire x1="83.5" y1="5.5" x2="82.0522" y2="6.9478" width="0.254" layer="16"/>
-<wire x1="81.27" y1="6.9478" x2="82.0522" y2="6.9478" width="0.254" layer="16"/>
+<wire x1="80.77" y1="6.897" x2="82.103" y2="6.897" width="0.25" layer="16"/>
+<wire x1="82.103" y1="6.897" x2="83.5" y2="5.5" width="0.25" layer="16"/>
 </signal>
 <signal name="STATUS_LED">
@@
 <contactref element="JP4" pad="8"/>
 <contactref element="JP7" pad="2"/>
-<wire x1="86.81" y1="6.9478" x2="87.7922" y2="6.9478" width="0.254" layer="16"/>
-<wire x1="87.7922" y1="6.9478" x2="89.66" y2="5.08" width="0.254" layer="16"/>
 <wire x1="89.66" y1="5.08" x2="89.66" y2="3.81" width="0.254" layer="16"/>
 <wire x1="89.66" y1="3.81" x2="90.93" y2="2.54" width="0.254" layer="16"/>
@@
 <wire x1="102.5" y1="4.103" x2="102.5" y2="3.95" width="0.254" layer="16"/>
 <wire x1="102.5" y1="3.95" x2="101.09" y2="2.54" width="0.254" layer="16"/>
+<wire x1="86.81" y1="6.897" x2="87.843" y2="6.897" width="0.25" layer="16"/>
+<wire x1="87.843" y1="6.897" x2="89.66" y2="5.08" width="0.25" layer="16"/>
 </signal>
 <signal name="BT">
